Commit message: change-05

File: src/amr_simulation/models/amr.xacro (robot description, xacro)
@@ -3,12 +3,7 @@
   AMR Description (Xacro)
   Differential-drive mobile robot with parameterized prefix for multi-robot namespacing.
-  Features:
-    - Base footprint and chassis link (0.6m x 0.5m x 0.2m)
-    - Left and right differential drive wheels (0.1m radius)
-    - Front and rear passive caster wheels
-    - 2D LiDAR ray sensor plugin (360 deg FOV, 10m range, 10 Hz)
-    - Gazebo differential drive plugin publishing odometry and wheel transforms
 -->
 <robot xmlns:xacro="http://www.ros.org/wiki/xacro" name="amr">
+    <!-- IMPORTANT: Assumes robot_name is passed WITH a trailing slash from the launch file (e.g., 'amr1/') -->
     <xacro:arg name="robot_name" default=""/>
     <link name="$(arg robot_name)base_footprint"/>
@@ -33,4 +28,6 @@
         </collision>
         <inertial>
+            <!-- FIX: Shifted Center of Mass forward by 0.1m to prevent backward tipping -->
+            <origin xyz="0.1 0 0" rpy="0 0 0"/>
             <mass value="10.0"/>
             <inertia ixx="0.24" ixy="0" ixz="0" iyy="0.33" iyz="0" izz="0.5"/>
@@ -67,5 +64,5 @@
     <xacro:wheel side="left" y_reflect="1"/>
     <xacro:wheel side="right" y_reflect="-1"/>
-    <!-- Caster wheel to keep it stable -->
+    <!-- Front Caster wheel -->
     <link name="$(arg robot_name)caster_wheel">
         <visual>
@@ -122,4 +119,6 @@
             <topic>/$(arg robot_name)scan</topic>
             <gz_frame_id>$(arg robot_name)lidar_link</gz_frame_id>
+            <!-- FIX: Added explicit ROS 2 frame ID -->
+            <frame_id>$(arg robot_name)lidar_link</frame_id>
             <ray>
                 <scan>
@@ -145,6 +144,7 @@
     </gazebo>
     <gazebo reference="$(arg robot_name)caster_wheel">
-        <mu1 value="0.001"/>
-        <mu2 value="0.001"/>
+        <!-- FIX: Corrected Gazebo SDF friction parameter syntax -->
+        <mu1>0.001</mu1>
+        <mu2>0.001</mu2>
     </gazebo>
     <gazebo>

Commit message: navigate to choke point done

File: src/amr_simulation/models/amr.xacro (robot description, xacro)
@@ -97,9 +97,4 @@
             </material>
         </visual>
-        <collision>
-            <geometry>
-                <cylinder radius="0.05" length="0.05"/>
-            </geometry>
-        </collision>
         <inertial>
             <mass value="0.1"/>
